File: AMP Projects/Mid 2x 35W AMP/2x35W AMP 1.6in x 1.2in.brd (EAGLE design)
At the start: 31.1 x 49.5 mm, 18 parts

Commit message: Updates to most boards
Parts:
- removed GND/CLIP, IN, OUT1, OUT3: M023.5MM, SparkFun-Connectors:SCREWTERMINAL-3.5MM-2
- removed PLUS/MINUS/GND: (no value), SparkFun-Connectors:SCREWTERMINAL-3.5MM-3
- removed ST-BY: M01PTH_2MM, SparkFun-Connectors:1X01_2MM
- added JP1, JP5: (no value), SparkFun-Connectors:1X05-1MM-RA
- added JP2, JP4: (no value), SparkFun-Connectors:1X04-1MM-RA
- moved R1 4.49 mm to (17.8, 7.62)
- moved C1 0.63 mm to (9.53, 10.8)
Connections:
- removed net N$8: R1.P$1, ST-BY.1
- new net +5V: JP1.2, JP4.4, JP5.2
- new net ST-BY: JP5.5, R1.P$1
- net CLIP: now also JP1.5; no longer GND/CLIP.2
- net GND: now also JP1.1, JP4.1, JP4.3, JP5.1; no longer GND/CLIP.1, PLUS/MINUS/GND.2, PLUS/MINUS/GND.3
- net OUT1: now also JP2.4; no longer OUT1.1
- net OUT2: now also JP2.3; no longer OUT1.2
- net OUT3: now also JP2.2; no longer OUT3.1
- net OUT4: now also JP2.1; no longer OUT3.2
- net RAW_IN1: now also JP1.4, JP5.4; no longer IN.2
- net RAW_IN3: now also JP1.3, JP5.3; no longer IN.1
- net VCC: now also JP4.2; no longer PLUS/MINUS/GND.1
Routing:
- net GND: track 122.4 -> 0.00 mm, vias 5 -> 0
- net CLIP: track 83.1 -> 0.00 mm
- net OUT4: track 41.7 -> 0.00 mm, vias 2 -> 0
- net OUT3: track 31.8 -> 0.00 mm
- net OUT2: track 23.5 -> 0.00 mm
- net N$8: track 19.5 -> 0.00 mm
- net OUT1: track 19.0 -> 0.00 mm
- net RAW_IN3: track 32.4 -> 20.4 mm
- net RAW_IN1: track 9.77 -> 0.00 mm
- net N$1: track 37.5 -> 41.9 mm
- net VCC: track 63.7 -> 59.6 mm
- net IN1: track 32.5 -> 33.2 mm
Other:
- board text removed: "1"
- board text removed: "2"
