File: AMP Projects/Mid 2x 35W AMP/2x35W AMP 1.6in x 1.2in.sch (EAGLE design)
At the start: 14 parts

Commit message: Updates to most boards
Parts:
- removed GND/CLIP, IN, OUT1, OUT3: M023.5MM, SparkFun-Connectors:M023.5MM
- removed PLUS/MINUS/GND: (no value), SparkFun-Connectors:M03SCREW
- removed ST-BY: M01PTH_2MM, SparkFun-Connectors:M01PTH_2MM
- added JP1, JP5: (no value), SparkFun-Connectors:M05SMD2
- added JP2, JP4: (no value), SparkFun-Connectors:M04SMD2
Connections:
- removed net N$8: R1.1, ST-BY.1
- new net +5V: JP1.2, JP4.4, JP5.2
- new net ST-BY: JP5.5, R1.1
- net CLIP: now also JP1.5; no longer GND/CLIP.2
- net GND: now also JP1.1, JP4.1, JP4.3, JP5.1; no longer GND/CLIP.1, PLUS/MINUS/GND.2, PLUS/MINUS/GND.3
- net OUT1: now also JP2.4; no longer OUT1.1
- net OUT2: now also JP2.3; no longer OUT1.2
- net OUT3: now also JP2.2; no longer OUT3.1
- net OUT4: now also JP2.1; no longer OUT3.2
- net RAW_IN1: now also JP1.4, JP5.4; no longer IN.2
- net RAW_IN3: now also JP1.3, JP5.3; no longer IN.1
- net VCC: now also JP4.2; no longer PLUS/MINUS/GND.1
Changed lines of the file:
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@@
 <?xml version="1.0" encoding="utf-8"?>
 <!DOCTYPE eagle SYSTEM "eagle.dtd">
-<eagle version="6.5.0">
+<eagle version="7.1.0">
 <drawing>
 <settings>
@@
 <part name="C3" library="SparkFun-Passives" deviceset="CAP" device="1206" value=".1uF"/>
 <part name="R1" library="SparkFun-Passives" deviceset="RESISTOR" device="PTH-1/4W" value="10k"/>
-<part name="ST-BY" library="SparkFun-Connectors" deviceset="M01" device="PTH_2MM"/>
-<part name="OUT1" library="SparkFun-Connectors" deviceset="M02" device="3.5MM" value="M023.5MM"/>
-<part name="OUT3" library="SparkFun-Connectors" deviceset="M02" device="3.5MM" value="M023.5MM"/>
-<part name="IN" library="SparkFun-Connectors" deviceset="M02" device="3.5MM" value="M023.5MM"/>
-<part name="GND/CLIP" library="SparkFun-Connectors" deviceset="M02" device="3.5MM" value="M023.5MM"/>
-<part name="PLUS/MINUS/GND" library="SparkFun-Connectors" deviceset="M03" device="SCREW"/>
+<part name="JP2" library="SparkFun-Connectors" deviceset="M04" device="SMD2"/>
+<part name="JP1" library="SparkFun-Connectors" deviceset="M05" device="SMD2"/>
+<part name="JP4" library="SparkFun-Connectors" deviceset="M04" device="SMD2"/>
+<part name="JP5" library="SparkFun-Connectors" deviceset="M05" device="SMD2"/>
 </parts>
 <sheets>
@@
 <instance part="C3" gate="G$1" x="55.88" y="30.48" rot="R90"/>
 <instance part="R1" gate="G$1" x="-2.54" y="58.42"/>
-<instance part="ST-BY" gate="G$1" x="-17.78" y="58.42"/>
-<instance part="OUT1" gate="G$1" x="137.16" y="83.82" rot="R180"/>
-<instance part="OUT3" gate="G$1" x="137.16" y="71.12" rot="R180"/>
-<instance part="IN" gate="G$1" x="-25.4" y="76.2"/>
-<instance part="GND/CLIP" gate="G$1" x="25.4" y="106.68" rot="R270"/>
-<instance part="PLUS/MINUS/GND" gate="G$1" x="55.88" y="2.54" rot="R90"/>
+<instance part="JP2" gate="G$1" x="139.7" y="76.2" rot="MR0"/>
+<instance part="JP1" gate="G$1" x="-30.48" y="101.6"/>
+<instance part="JP4" gate="G$1" x="55.88" y="0" rot="R90"/>
+<instance part="JP5" gate="G$1" x="-30.48" y="76.2"/>
 </instances>
 <busses>
@@
 <wire x1="81.28" y1="30.48" x2="58.42" y2="30.48" width="0.1524" layer="91"/>
 <wire x1="58.42" y1="30.48" x2="58.42" y2="22.86" width="0.1524" layer="91"/>
-<wire x1="58.42" y1="22.86" x2="58.42" y2="10.16" width="0.1524" layer="91"/>
+<wire x1="58.42" y1="22.86" x2="58.42" y2="15.24" width="0.1524" layer="91"/>
 <junction x="58.42" y="22.86"/>
 <junction x="58.42" y="30.48"/>
-<pinref part="PLUS/MINUS/GND" gate="G$1" pin="1"/>
+</segment>
+<segment>
+<pinref part="JP4" gate="G$1" pin="2"/>
+<wire x1="55.88" y1="5.08" x2="55.88" y2="10.16" width="0.1524" layer="91"/>
+<label x="55.88" y="5.08" size="1.778" layer="95" rot="R90"/>
 </segment>
 </net>
@@
 <wire x1="50.8" y1="30.48" x2="27.94" y2="30.48" width="0.1524" layer="91"/>
 <wire x1="27.94" y1="30.48" x2="27.94" y2="43.18" width="0.1524" layer="91"/>
-<wire x1="50.8" y1="22.86" x2="50.8" y2="12.7" width="0.1524" layer="91"/>
+<wire x1="50.8" y1="22.86" x2="50.8" y2="15.24" width="0.1524" layer="91"/>
 <junction x="50.8" y="22.86"/>
 <junction x="50.8" y="30.48"/>
-<wire x1="50.8" y1="12.7" x2="53.34" y2="12.7" width="0.1524" layer="91"/>
-<pinref part="PLUS/MINUS/GND" gate="G$1" pin="3"/>
-<wire x1="53.34" y1="12.7" x2="53.34" y2="10.16" width="0.1524" layer="91"/>
-</segment>
-<segment>
-<pinref part="GND/CLIP" gate="G$1" pin="1"/>
-<wire x1="25.4" y1="99.06" x2="25.4" y2="91.44" width="0.1524" layer="91"/>
+<wire x1="50.8" y1="15.24" x2="53.34" y2="15.24" width="0.1524" layer="91"/>
+<pinref part="JP4" gate="G$1" pin="3"/>
+<wire x1="53.34" y1="5.08" x2="53.34" y2="15.24" width="0.1524" layer="91"/>
+<label x="53.34" y="5.08" size="1.778" layer="95" rot="R90"/>
 </segment>
 <segment>
@@
 </segment>
 <segment>
-<pinref part="PLUS/MINUS/GND" gate="G$1" pin="2"/>
-<wire x1="55.88" y1="10.16" x2="55.88" y2="15.24" width="0.1524" layer="91"/>
-<label x="53.34" y="15.24" size="1.778" layer="95"/>
-</segment>
-</net>
-<net name="N$8" class="0">
+<pinref part="JP4" gate="G$1" pin="1"/>
+<wire x1="58.42" y1="5.08" x2="58.42" y2="10.16" width="0.1524" layer="91"/>
+<label x="58.42" y="5.08" size="1.778" layer="95" rot="R90"/>
+</segment>
+<segment>
+<wire x1="-22.86" y1="71.12" x2="-17.78" y2="71.12" width="0.1524" layer="91"/>
+<label x="-22.86" y="71.12" size="1.778" layer="95"/>
+<pinref part="JP5" gate="G$1" pin="1"/>
+</segment>
+<segment>
+<pinref part="JP1" gate="G$1" pin="1"/>
+<wire x1="-22.86" y1="96.52" x2="-10.16" y2="96.52" width="0.1524" layer="91"/>
+<label x="-17.78" y="96.52" size="1.778" layer="95"/>
+</segment>
+</net>
+<net name="ST-BY" class="0">
 <segment>
 <pinref part="R1" gate="G$1" pin="1"/>
 <wire x1="-7.62" y1="58.42" x2="-10.16" y2="58.42" width="0.1524" layer="91"/>
-<pinref part="ST-BY" gate="G$1" pin="1"/>
+</segment>
+<segment>
+<wire x1="-22.86" y1="81.28" x2="-17.78" y2="81.28" width="0.1524" layer="91"/>
+<label x="-20.32" y="81.28" size="1.778" layer="95"/>
+<pinref part="JP5" gate="G$1" pin="5"/>
 </segment>
 </net>
@@
 <segment>
 <pinref part="U$1" gate="G$1" pin="OUT4"/>
-<pinref part="OUT3" gate="G$1" pin="2"/>
 <wire x1="81.28" y1="68.58" x2="129.54" y2="68.58" width="0.1524" layer="91"/>
+<wire x1="129.54" y1="68.58" x2="129.54" y2="73.66" width="0.1524" layer="91"/>
+<pinref part="JP2" gate="G$1" pin="1"/>
+<wire x1="129.54" y1="73.66" x2="134.62" y2="73.66" width="0.1524" layer="91"/>
 </segment>
 </net>
@@
 <segment>
 <pinref part="U$1" gate="G$1" pin="OUT2"/>
-<wire x1="81.28" y1="78.74" x2="116.84" y2="78.74" width="0.1524" layer="91"/>
-<wire x1="116.84" y1="78.74" x2="116.84" y2="81.28" width="0.1524" layer="91"/>
-<pinref part="OUT1" gate="G$1" pin="2"/>
-<wire x1="116.84" y1="81.28" x2="129.54" y2="81.28" width="0.1524" layer="91"/>
+<wire x1="81.28" y1="78.74" x2="134.62" y2="78.74" width="0.1524" layer="91"/>
+<pinref part="JP2" gate="G$1" pin="3"/>
 </segment>
 </net>
@@
 <pinref part="U$1" gate="G$1" pin="OUT1"/>
 <wire x1="129.54" y1="83.82" x2="81.28" y2="83.82" width="0.1524" layer="91"/>
-<pinref part="OUT1" gate="G$1" pin="1"/>
+<wire x1="129.54" y1="83.82" x2="129.54" y2="81.28" width="0.1524" layer="91"/>
+<pinref part="JP2" gate="G$1" pin="4"/>
+<wire x1="129.54" y1="81.28" x2="134.62" y2="81.28" width="0.1524" layer="91"/>
 </segment>
 </net>
@@
 <wire x1="-10.16" y1="83.82" x2="15.24" y2="83.82" width="0.1524" layer="91"/>
 <label x="2.54" y="83.82" size="1.778" layer="95"/>
-<pinref part="IN" gate="G$1" pin="2"/>
-<wire x1="-17.78" y1="78.74" x2="-10.16" y2="78.74" width="0.1524" layer="91"/>
 <wire x1="-10.16" y1="78.74" x2="-10.16" y2="83.82" width="0.1524" layer="91"/>
+<wire x1="-10.16" y1="78.74" x2="-22.86" y2="78.74" width="0.1524" layer="91"/>
+<pinref part="JP5" gate="G$1" pin="4"/>
+</segment>
+<segment>
+<pinref part="JP1" gate="G$1" pin="4"/>
+<wire x1="-22.86" y1="104.14" x2="-10.16" y2="104.14" width="0.1524" layer="91"/>
+<label x="-17.78" y="104.14" size="1.778" layer="95"/>
 </segment>
 </net>
@@
 <pinref part="C2" gate="G$1" pin="2"/>
 <label x="5.08" y="73.66" size="1.778" layer="95"/>
-<pinref part="IN" gate="G$1" pin="1"/>
-<wire x1="-17.78" y1="76.2" x2="-10.16" y2="76.2" width="0.1524" layer="91"/>
 <wire x1="-10.16" y1="76.2" x2="-10.16" y2="73.66" width="0.1524" layer="91"/>
 <wire x1="-10.16" y1="73.66" x2="15.24" y2="73.66" width="0.1524" layer="91"/>
+<wire x1="-10.16" y1="76.2" x2="-22.86" y2="76.2" width="0.1524" layer="91"/>
+<pinref part="JP5" gate="G$1" pin="3"/>
+</segment>
+<segment>
+<pinref part="JP1" gate="G$1" pin="3"/>
+<wire x1="-22.86" y1="101.6" x2="-10.16" y2="101.6" width="0.1524" layer="91"/>
+<label x="-17.78" y="101.6" size="1.778" layer="95"/>
 </segment>
 </net>
@@
 <pinref part="U$1" gate="G$1" pin="DIAGNOSTICS"/>
 <wire x1="81.28" y1="58.42" x2="86.36" y2="58.42" width="0.1524" layer="91"/>
-</segment>
-<segment>
-<pinref part="GND/CLIP" gate="G$1" pin="2"/>
-<wire x1="27.94" y1="99.06" x2="27.94" y2="91.44" width="0.1524" layer="91"/>
+<label x="83.82" y="58.42" size="1.778" layer="95"/>
+</segment>
+<segment>
+<pinref part="JP1" gate="G$1" pin="5"/>
+<wire x1="-22.86" y1="106.68" x2="-12.7" y2="106.68" width="0.1524" layer="91"/>
+<wire x1="-10.16" y1="106.68" x2="-12.7" y2="106.68" width="0.1524" layer="91"/>
+<label x="-17.78" y="106.68" size="1.778" layer="95"/>
 </segment>
 </net>
@@
 <pinref part="U$1" gate="G$1" pin="OUT3"/>
 <wire x1="116.84" y1="73.66" x2="81.28" y2="73.66" width="0.1524" layer="91"/>
-<wire x1="116.84" y1="73.66" x2="116.84" y2="71.12" width="0.1524" layer="91"/>
-<pinref part="OUT3" gate="G$1" pin="1"/>
-<wire x1="116.84" y1="71.12" x2="129.54" y2="71.12" width="0.1524" layer="91"/>
-</segment>
-</net>
+<wire x1="116.84" y1="73.66" x2="116.84" y2="76.2" width="0.1524" layer="91"/>
+<pinref part="JP2" gate="G$1" pin="2"/>
+<wire x1="116.84" y1="76.2" x2="134.62" y2="76.2" width="0.1524" layer="91"/>
+</segment>
+</net>
+<net name="+5V" class="0">
+<segment>
+<pinref part="JP4" gate="G$1" pin="4"/>
+<wire x1="50.8" y1="5.08" x2="50.8" y2="10.16" width="0.1524" layer="91"/>
+<label x="50.8" y="5.08" size="1.778" layer="95" rot="R90"/>
+</segment>
+<segment>
+<pinref part="JP1" gate="G$1" pin="2"/>
+<wire x1="-22.86" y1="99.06" x2="-10.16" y2="99.06" width="0.1524" layer="91"/>
+<label x="-17.78" y="99.06" size="1.778" layer="95"/>
+</segment>
+<segment>
+<pinref part="JP5" gate="G$1" pin="2"/>
+<wire x1="-22.86" y1="73.66" x2="-17.78" y2="73.66" width="0.1524" layer="91"/>
+<label x="-20.32" y="73.66" size="1.778" layer="95"/>
+</segment>
+</net>
