File: AMP Projects/VU Meter/VU Meter 1inchx3inches V1.0.sch (EAGLE design)
At the start: 19 parts, among them IC1 LM3914N

Commit message: Updates to most boards
Parts:
- removed CLIP+, CLIP-, SIGIN: M01PTH, SparkFun-Connectors:M01PTH
- removed G1: AB9V, battery:AB9V
- removed S1: (no value), switch-omron:10-XX
- added CLIP1, LED11, LED12, LED13, LED14, LED15, LED16, LED17, LED18, LED19, LED20: (no value), led:LED5MM
- added IC2: LM3914N, national-semiconductor:LM3914N
- added JP1: (no value), SparkFun-Connectors:M05SMD2
- added R3: 3300, SparkFun-Resistors:RESISTORPTH-1/4W
- added R4: 2200, SparkFun-Resistors:RESISTORPTH-1/4W
- added S2: (no value), switch-omron:10-XX
Connections:
- removed net N$15: IC1.MODE, S1.P, S1.P1
- new net CLIP+: CLIP.A, CLIP1.A, JP1.5
- new net L-SIG: IC1.SIGIN, JP1.3
- new net MODE: IC1.MODE, IC2.MODE, S2.P, S2.P1
- new net N$14: IC2.REFOUT, IC2.RHI, R4.1
- new net N$19: IC2.LED4, LED14.C
- new net N$20: IC2.LED5, LED15.C
- new net N$21: IC2.LED6, LED16.C
- new net N$23: IC2.LED7, LED17.C
- new net N$24: IC2.LED8, LED18.C
- new net N$25: IC2.LED9, LED19.C
- new net N$26: IC2.LED10, LED20.C
- new net N$27: IC2.REFADJ, R3.2, R4.2
- new net R-SIG: IC2.SIGIN, JP1.4
- net GND: now also CLIP.C, CLIP1.C, IC2.RLO, IC2.V-, JP1.1, R3.1; no longer G1.-
- net N$16: now also IC2.LED1, LED11.C; no longer IC1.SIGIN, SIGIN.1
- net N$17: now also IC2.LED2, LED12.C; no longer CLIP+.1, CLIP.A
- net N$18: now also IC2.LED3, LED13.C; no longer CLIP-.1, CLIP.C
- net V+: now also IC2.V+, JP1.2, LED11.A, LED12.A, LED13.A, LED14.A, LED15.A, LED16.A, LED17.A, LED18.A, LED19.A, LED20.A, S2.S, S2.S1; no longer G1.+, S1.S, S1.S1
Other:
- moved on the sheet: CLIP
