File: AMP Projects/VU Meter Integrator/integrator.brd (EAGLE design)
At the start: 41.9 x 54 mm, 32 parts, among them IC1 OPAMP-DUALDIP

Commit message: Updates to most boards
Parts:
- removed IN, OUT, PWR_IN, PWR_PARALLEL: M023.5MM, SparkFun-Connectors:SCREWTERMINAL-3.5MM-2
- added JP1, JP2: (no value), SparkFun-Connectors:1X05-1MM-RA
- moved R10 7.65 mm to (8.89, 45.1)
- moved R7 7.65 mm to (8.89, 47.6)
- moved R8 0.63 mm to (29.2, 45.1)
- moved R9 0.63 mm to (29.2, 47.6)
Connections:
- new net CLIP+: JP1.5, JP2.5
- net 5V: now also JP1.2, JP2.2; no longer PWR_IN.1, PWR_PARALLEL.2
- net GND: now also JP1.1, JP2.1; no longer PWR_IN.2, PWR_PARALLEL.1
- net L_IN: now also JP1.3; no longer IN.2
- net L_OUT: now also JP2.3; no longer OUT.1
- net R_IN: now also JP1.4; no longer IN.1
- net R_OUT: now also JP2.4; no longer OUT.2
Routing:
- net GND: track 103.2 -> 0.00 mm, vias 11 -> 8
- net CLIP+: track 0.00 -> 78.6 mm, vias 0 -> 2
- net 5V: track 29.7 -> 49.1 mm
- net L_OUT: track 41.0 -> 28.1 mm
- net R_OUT: track 37.1 -> 26.5 mm
- net N$12: track 7.40 -> 15.9 mm
- net L_IN: track 12.3 -> 19.1 mm
- net N$2: track 30.6 -> 26.3 mm
- net R_IN: track 12.2 -> 13.7 mm, vias 0 -> 1
- net N$13: track 18.3 -> 17.7 mm
Other:
- outline, holes or cut-outs redrawn
