File: AMP Projects/Input module/input module.brd (EAGLE design)
At the start: 43.2 x 36.8 mm, 20 parts, among them IC1 OPAMP-DUALU

Commit message: Fixed incorrect usage of op-amp on pre-amplifier.
Parts:
- moved C4 5.46 mm to (19.7, 12.7)
- moved C1 0.64 mm to (26.0, 18.4)
Connections:
- net GND: now also IC1.5; no longer IC1.6
- net N$3: now also IC1.6; no longer IC1.5
Routing:
- net GND: track 70.2 -> 57.1 mm, vias 8 -> 9
- net N$5: track 34.7 -> 43.2 mm
- net N$3: track 20.5 -> 22.0 mm
- net +V: track 21.9 -> 22.4 mm
Changed lines of the file:
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@@
 <?xml version="1.0" encoding="utf-8"?>
 <!DOCTYPE eagle SYSTEM "eagle.dtd">
-<eagle version="6.5.0">
+<eagle version="7.7.0">
 <drawing>
 <settings>
@@
 <pass name="Default">
 <param name="RoutingGrid" value="50mil"/>
+<param name="AutoGrid" value="1"/>
+<param name="Efforts" value="0"/>
+<param name="TopRouterVariant" value="1"/>
 <param name="tpViaShape" value="round"/>
 <param name="PrefDir.1" value="|"/>
@@
 <element name="RV3" library="SparkFun-Electromechanical" package="ALPS_POT" value="20k" x="29.21" y="32.385" rot="R270"/>
 <element name="RV4" library="SparkFun-Electromechanical" package="ALPS_POT" value="20k" x="8.89" y="32.385" rot="R270"/>
-<element name="C1" library="SparkFun-Capacitors" package="1206" value="100nF" x="25.4" y="18.415" rot="R270"/>
+<element name="C1" library="SparkFun-Capacitors" package="1206" value="100nF" x="26.035" y="18.415" rot="R270"/>
 <element name="C2" library="SparkFun-Capacitors" package="1206" value="100nF" x="10.16" y="15.875" rot="R270"/>
 <element name="C3" library="SparkFun-Passives" package="0805" value="47pF" x="12.065" y="19.685" rot="R90"/>
-<element name="C4" library="SparkFun-Passives" package="0805" value="47pF" x="22.86" y="17.145" rot="R90"/>
+<element name="C4" library="SparkFun-Passives" package="0805" value="47pF" x="19.685" y="12.7" rot="R90"/>
 <element name="RV1" library="SparkFun-Electromechanical" package="TRIM_POT" value="100K" x="1.27" y="15.24"/>
 <element name="RV2" library="SparkFun-Electromechanical" package="TRIM_POT" value="100K" x="34.29" y="20.32" rot="R180"/>
@@
 <contactref element="JP1" pad="2"/>
 <contactref element="RV4" pad="P$3"/>
-<contactref element="IC1" pad="6"/>
 <wire x1="10.16" y1="17.275" x2="9.655" y2="17.275" width="0.4064" layer="1"/>
 <wire x1="9.655" y1="17.275" x2="8.255" y2="15.875" width="0.4064" layer="1"/>
@@
 <wire x1="31.75" y1="20.32" x2="28.575" y2="17.145" width="0.4064" layer="16"/>
 <via x="28.575" y="17.145" extent="1-16" drill="0.6" shape="square"/>
-<wire x1="28.575" y1="17.145" x2="25.53" y2="17.145" width="0.4064" layer="1"/>
-<wire x1="25.53" y1="17.145" x2="25.4" y2="17.015" width="0.4064" layer="1"/>
-<wire x1="25.4" y1="17.015" x2="25.4" y2="17.145" width="0.4064" layer="1"/>
-<wire x1="25.4" y1="17.145" x2="22.225" y2="17.145" width="0.3048" layer="1"/>
-<wire x1="22.225" y1="17.145" x2="20.955" y2="17.78" width="0.3048" layer="1"/>
-<wire x1="20.955" y1="17.78" x2="20.3962" y2="17.78" width="0.4064" layer="1"/>
-<wire x1="15.1638" y1="17.78" x2="20.3962" y2="17.78" width="0.4064" layer="1"/>
+<wire x1="25.53" y1="17.145" x2="26.035" y2="17.015" width="0.4064" layer="1"/>
+<wire x1="26.035" y1="17.015" x2="26.035" y2="17.145" width="0.4064" layer="1"/>
 <wire x1="18.09" y1="4.445" x2="18.09" y2="4.12" width="0.4064" layer="1"/>
 <wire x1="18.09" y1="4.12" x2="16.51" y2="2.54" width="0.4064" layer="1"/>
@@
 <via x="20.32" y="32.385" extent="1-16" drill="0.6" shape="square"/>
 <via x="36.195" y="27.94" extent="1-16" drill="0.6" shape="square"/>
+<contactref element="IC1" pad="5"/>
+<via x="20.955" y="15.24" extent="1-16" drill="0.6" shape="square"/>
 </signal>
 <signal name="+V">
@@
 <wire x1="20.3962" y1="20.32" x2="23.495" y2="20.32" width="0.4064" layer="1"/>
 <wire x1="23.495" y1="20.32" x2="24.895" y2="20.32" width="0.4064" layer="1"/>
-<wire x1="24.895" y1="20.32" x2="25.4" y2="19.815" width="0.4064" layer="1"/>
+<wire x1="24.895" y1="20.32" x2="26.035" y2="19.815" width="0.4064" layer="1"/>
 <wire x1="21.59" y1="4.445" x2="21.59" y2="7.62" width="0.4064" layer="1"/>
 <wire x1="21.59" y1="7.62" x2="23.495" y2="9.525" width="0.4064" layer="1"/>
@@
 <wire x1="15.24" y1="27.94" x2="15.24" y2="24.13" width="0.4064" layer="1"/>
 <wire x1="15.24" y1="24.13" x2="18.415" y2="24.13" width="0.4064" layer="1"/>
-<wire x1="18.415" y1="24.13" x2="18.415" y2="19.05" width="0.4064" layer="1"/>
+<wire x1="18.415" y1="24.13" x2="18.415" y2="22.225" width="0.4064" layer="1"/>
+<wire x1="18.415" y1="22.225" x2="18.415" y2="19.05" width="0.4064" layer="1"/>
 <wire x1="18.415" y1="19.05" x2="20.3962" y2="19.05" width="0.4064" layer="1"/>
-<wire x1="22.86" y1="18.045" x2="23.125" y2="18.045" width="0.4064" layer="1"/>
-<wire x1="23.125" y1="18.045" x2="24.13" y2="18.415" width="0.4064" layer="1"/>
-<wire x1="24.13" y1="18.415" x2="27.305" y2="18.415" width="0.4064" layer="1"/>
-<wire x1="27.305" y1="18.415" x2="29.21" y2="20.32" width="0.4064" layer="1"/>
-<wire x1="20.3962" y1="19.05" x2="21.22" y2="19.05" width="0.4064" layer="1"/>
-<wire x1="21.22" y1="19.05" x2="22.86" y2="18.045" width="0.4064" layer="1"/>
+<wire x1="19.685" y1="13.6" x2="18.785" y2="13.6" width="0.4064" layer="1"/>
+<wire x1="18.785" y1="13.6" x2="18.415" y2="13.97" width="0.4064" layer="1"/>
+<wire x1="18.415" y1="13.97" x2="18.415" y2="19.05" width="0.4064" layer="1"/>
+<wire x1="29.21" y1="20.32" x2="29.21" y2="20.955" width="0.4064" layer="1"/>
+<wire x1="29.21" y1="20.955" x2="27.94" y2="22.225" width="0.4064" layer="1"/>
+<wire x1="27.94" y1="22.225" x2="18.415" y2="22.225" width="0.4064" layer="1"/>
 </signal>
 <signal name="N$3">
 <contactref element="C4" pad="1"/>
 <contactref element="R2" pad="P$1"/>
+<wire x1="19.685" y1="11.8" x2="23.125" y2="14.975" width="0.4064" layer="1"/>
+<wire x1="23.125" y1="14.975" x2="25.4" y2="14.605" width="0.4064" layer="1"/>
 <contactref element="R4" pad="P$2"/>
-<contactref element="IC1" pad="5"/>
-<wire x1="10.16" y1="12.065" x2="20.3962" y2="12.065" width="0.4064" layer="1"/>
-<wire x1="20.3962" y1="12.065" x2="20.3962" y2="15.875" width="0.4064" layer="1"/>
-<wire x1="20.3962" y1="15.875" x2="20.3962" y2="16.51" width="0.4064" layer="1"/>
-<wire x1="22.86" y1="16.245" x2="23.76" y2="16.245" width="0.4064" layer="1"/>
-<wire x1="23.76" y1="16.245" x2="25.4" y2="14.605" width="0.4064" layer="1"/>
-<wire x1="22.86" y1="16.245" x2="22.595" y2="16.245" width="0.4064" layer="1"/>
-<wire x1="22.595" y1="16.245" x2="22.225" y2="15.875" width="0.4064" layer="1"/>
-<wire x1="22.225" y1="15.875" x2="20.3962" y2="15.875" width="0.4064" layer="1"/>
+<contactref element="IC1" pad="6"/>
+<wire x1="16.51" y1="12.065" x2="10.16" y2="12.065" width="0.4064" layer="1"/>
+<wire x1="19.685" y1="11.8" x2="16.775" y2="11.8" width="0.4064" layer="1"/>
+<wire x1="16.775" y1="11.8" x2="16.51" y2="12.065" width="0.4064" layer="1"/>
+<wire x1="23.125" y1="14.975" x2="22.86" y2="15.24" width="0.4064" layer="1"/>
+<wire x1="22.86" y1="15.24" x2="22.86" y2="17.78" width="0.4064" layer="1"/>
+<wire x1="22.86" y1="17.78" x2="20.3962" y2="17.78" width="0.4064" layer="1"/>
 </signal>
 <signal name="R_IN">
